Commit message: urdf
Signed-off-by: adrianCo <adrian.cobo.mh@gmail.com>

File: description/soporte_core.xacro (robot description, xacro)
@@ -41,24 +41,24 @@
         <origin xyz="1.0 0.0 0.0" rpy="0.0 0.0 0.0"/>
         <parent link="base_chassis"/>
-        <child link="base_c1"/>
+        <child link="oak1_rgb_camera_optical_frame"/>
     </joint>
-    <link name="base_c1"></link>
+    <link name="oak1_rgb_camera_optical_frame"></link>
     <joint name="c2_joint" type="fixed">
         <origin xyz="0.0 1.0 0.0" rpy="0.0 0.0 ${pi/2}"/>
         <parent link="base_chassis"/>
-        <child link="base_c2"/>
+        <child link="oak2_rgb_camera_optical_frame"/>
     </joint>
-    <link name="base_c2"></link>
+    <link name="oak2_rgb_camera_optical_frame"></link>
     <joint name="c3_joint" type="fixed">
         <origin xyz="-1.0 0.0 0.0" rpy="0.0 0.0 ${pi}"/>
         <parent link="base_chassis"/>
-        <child link="base_c3"/>
+        <child link="oak3_rgb_camera_optical_frame"/>
     </joint>
-    <link name="base_c3"></link>
+    <link name="oak3_rgb_camera_optical_frame"></link>
     <joint name="c4_joint" type="fixed">
         <origin xyz="0.0 -1.0 0.0" rpy="0.0 0.0 ${3*pi/2}"/>
         <parent link="base_chassis"/>
-        <child link="base_c4"/>
+        <child link="oak4_rgb_camera_optical_frame"/>
     </joint>
-    <link name="base_c4"></link>
+    <link name="oak4_rgb_camera_optical_frame"></link>
 </robot>

Commit message: finish
Signed-off-by: adrianCo <adrian.cobo.mh@gmail.com>

File: description/soporte_core.xacro (robot description, xacro)
@@ -41,24 +41,24 @@
         <origin xyz="1.0 0.0 0.0" rpy="0.0 0.0 0.0"/>
         <parent link="base_chassis"/>
-        <child link="oak1_rgb_camera_optical_frame"/>
+        <child link="oak1-d-base-frame"/>
     </joint>
-    <link name="oak1_rgb_camera_optical_frame"></link>
+    <link name="oak1-d-base-frame"></link>
     <joint name="c2_joint" type="fixed">
         <origin xyz="0.0 1.0 0.0" rpy="0.0 0.0 ${pi/2}"/>
         <parent link="base_chassis"/>
-        <child link="oak2_rgb_camera_optical_frame"/>
+        <child link="oak2-d-base-frame"/>
     </joint>
-    <link name="oak2_rgb_camera_optical_frame"></link>
+    <link name="oak2-d-base-frame"></link>
     <joint name="c3_joint" type="fixed">
         <origin xyz="-1.0 0.0 0.0" rpy="0.0 0.0 ${pi}"/>
         <parent link="base_chassis"/>
-        <child link="oak3_rgb_camera_optical_frame"/>
+        <child link="oak3-d-base-frame"/>
     </joint>
-    <link name="oak3_rgb_camera_optical_frame"></link>
+    <link name="oak3-d-base-frame"></link>
     <joint name="c4_joint" type="fixed">
         <origin xyz="0.0 -1.0 0.0" rpy="0.0 0.0 ${3*pi/2}"/>
         <parent link="base_chassis"/>
-        <child link="oak4_rgb_camera_optical_frame"/>
+        <child link="oak4-d-base-frame"/>
     </joint>
-    <link name="oak4_rgb_camera_optical_frame"></link>
+    <link name="oak4-d-base-frame"></link>
 </robot>

Commit message: adding meshes
Signed-off-by: adrianCo <adrian.cobo.mh@gmail.com>

File: description/soporte_core.xacro (robot description, xacro)
@@ -23,5 +23,5 @@
             <origin xyz="0.0 0.0 0.0" rpy="0.0 0.0 0.0"/>
             <geometry>
-                <box size="0.105 0.105 0.073"/>
+                <mesh filename="package://perception_system_v2/meshes/box.dae"/>
             </geometry>
             <material name="white"/>
@@ -30,5 +30,5 @@
             <origin xyz="0 0.0 -0.005" rpy="0.0 0.0 0.0"/>
             <geometry>
-                <box size="0.105 0.105 0.073"/>
+                <mesh filename="package://perception_system_v2/meshes/box.dae"/>
             </geometry>
         </collision>
@@ -39,5 +39,5 @@
     </link>
     <joint name="c1_joint" type="fixed">
-        <origin xyz="1.0 0.0 0.0" rpy="0.0 0.0 0.0"/>
+        <origin xyz="0.10 0.0 0.0" rpy="0.0 0.0 0.0"/>
         <parent link="base_chassis"/>
         <child link="oak1-d-base-frame"/>
@@ -45,5 +45,5 @@
     <link name="oak1-d-base-frame"></link>
     <joint name="c2_joint" type="fixed">
-        <origin xyz="0.0 1.0 0.0" rpy="0.0 0.0 ${pi/2}"/>
+        <origin xyz="0.05 0.05 0.0" rpy="0.0 0.0 ${30*pi/180}"/>
         <parent link="base_chassis"/>
         <child link="oak2-d-base-frame"/>
@@ -51,5 +51,5 @@
     <link name="oak2-d-base-frame"></link>
     <joint name="c3_joint" type="fixed">
-        <origin xyz="-1.0 0.0 0.0" rpy="0.0 0.0 ${pi}"/>
+        <origin xyz="0.05 -0.05 0.0" rpy="0.0 0.0 ${330*pi/180}"/>
         <parent link="base_chassis"/>
         <child link="oak3-d-base-frame"/>
@@ -57,5 +57,5 @@
     <link name="oak3-d-base-frame"></link>
     <joint name="c4_joint" type="fixed">
-        <origin xyz="0.0 -1.0 0.0" rpy="0.0 0.0 ${3*pi/2}"/>
+        <origin xyz="-1.0 0.0 0.0" rpy="0.0 0.0 ${pi}"/>
         <parent link="base_chassis"/>
         <child link="oak4-d-base-frame"/>

Commit message: need reorientate and reduce peace
Signed-off-by: adrianCo <adrian.cobo.mh@gmail.com>

File: description/soporte_core.xacro (robot description, xacro)
@@ -21,14 +21,14 @@
     <link name="base_chassis">
         <visual name="">
-            <origin xyz="0.0 0.0 0.0" rpy="0.0 0.0 0.0"/>
+            <origin xyz="0.0 0.0 0.0" rpy="0.0 ${pi/2} 0.0"/>
             <geometry>
-                <mesh filename="package://perception_system_v2/meshes/box.dae"/>
+                <mesh filename="package://perception_system_v2/meshes/soporte_160grad.dae" scale="0.001 0.001 0.001"/>
             </geometry>
             <material name="white"/>
         </visual>
         <collision>
-            <origin xyz="0 0.0 -0.005" rpy="0.0 0.0 0.0"/>
+            <origin xyz="0 0.0 0.0" rpy="0.0 ${pi/2} 0.0"/>
             <geometry>
-                <mesh filename="package://perception_system_v2/meshes/box.dae"/>
+                <mesh filename="package://perception_system_v2/meshes/soporte_160grad.dae" scale="0.001 0.001 0.001"/>
             </geometry>
         </collision>

Commit message: end
Signed-off-by: adrianCo <adrian.cobo.mh@gmail.com>

File: description/soporte_core.xacro (robot description, xacro)
@@ -21,5 +21,5 @@
     <link name="base_chassis">
         <visual name="">
-            <origin xyz="0.0 0.0 0.0" rpy="0.0 ${pi/2} 0.0"/>
+            <origin xyz="0.0 0.0 0.0" rpy="${pi/2} 0.0 ${pi/2}"/>
             <geometry>
                 <mesh filename="package://perception_system_v2/meshes/soporte_160grad.dae" scale="0.001 0.001 0.001"/>
@@ -28,5 +28,5 @@
         </visual>
         <collision>
-            <origin xyz="0 0.0 0.0" rpy="0.0 ${pi/2} 0.0"/>
+            <origin xyz="0.0 0.0 0.0" rpy="${pi/2} ${pi/2} 0.0"/>
             <geometry>
                 <mesh filename="package://perception_system_v2/meshes/soporte_160grad.dae" scale="0.001 0.001 0.001"/>
@@ -39,5 +39,5 @@
     </link>
     <joint name="c1_joint" type="fixed">
-        <origin xyz="0.10 0.0 0.0" rpy="0.0 0.0 0.0"/>
+        <origin xyz="0.03420 0.0 0.0" rpy="0.0 0.0 0.0"/>
         <parent link="base_chassis"/>
         <child link="oak1-d-base-frame"/>
@@ -45,5 +45,5 @@
     <link name="oak1-d-base-frame"></link>
     <joint name="c2_joint" type="fixed">
-        <origin xyz="0.05 0.05 0.0" rpy="0.0 0.0 ${30*pi/180}"/>
+        <origin xyz="0.01710 0.09698 0.0" rpy="0.0 0.0 ${30*pi/180}"/>
         <parent link="base_chassis"/>
         <child link="oak2-d-base-frame"/>
@@ -51,5 +51,5 @@
     <link name="oak2-d-base-frame"></link>
     <joint name="c3_joint" type="fixed">
-        <origin xyz="0.05 -0.05 0.0" rpy="0.0 0.0 ${330*pi/180}"/>
+        <origin xyz="0.01710 -0.09698 0.0" rpy="0.0 0.0 ${330*pi/180}"/>
         <parent link="base_chassis"/>
         <child link="oak3-d-base-frame"/>

Commit message: works for 160 grad
Signed-off-by: adrianCo <adrian.cobo.mh@gmail.com>

File: description/soporte_core.xacro (robot description, xacro)
@@ -21,14 +21,14 @@
     <link name="base_chassis">
         <visual name="">
-            <origin xyz="0.0 0.0 0.0" rpy="${pi/2} 0.0 ${pi/2}"/>
+            <origin xyz="0.0 0.0 0.0" rpy="0.0 0.0 0.0"/>
             <geometry>
-                <mesh filename="package://perception_system_v2/meshes/soporte_160grad.dae" scale="0.001 0.001 0.001"/>
+                <mesh filename="package://perception_system_v2/meshes/soporte_160grad.dae"/>
             </geometry>
             <material name="white"/>
         </visual>
         <collision>
-            <origin xyz="0.0 0.0 0.0" rpy="${pi/2} ${pi/2} 0.0"/>
+            <origin xyz="0.0 0.0 0.0" rpy="0.0 0.0 0.0"/>
             <geometry>
-                <mesh filename="package://perception_system_v2/meshes/soporte_160grad.dae" scale="0.001 0.001 0.001"/>
+                <mesh filename="package://perception_system_v2/meshes/soporte_160grad.dae"/>
             </geometry>
         </collision>
