Commit message: new .xacros
Signed-off-by: adrianco <adrian.cobo.mh@gmail.com>

File: description/soporte.xacro (robot description, xacro)
@@ -2,8 +2,16 @@
 <robot xmlns:xacro="http://www.ros.org/wiki/xacro"  name="robot">
     <xacro:include filename="inertial_macros.xacro"/>
-    <xacro:include filename="soporte_core_hexag.xacro" />
-    <!-- <xacro:include filename="$(find realsense2_description)/urdf/_d435.urdf.xacro" /> -->
-    <!-- <xacro:sensor_d435 parent="camera_attachment_link" use_nominal_extrinsics="$(arg use_nominal_extrinsics)" add_plug="$(arg add_plug)" use_mesh="$(arg use_mesh)">
-        <origin xyz="0.075 0 -0.01" rpy="0 0 0"/>
-    </xacro:sensor_d435> -->
+    <xacro:include filename="soporte_core.xacro" />
+    <xacro:include filename="soporte_camera.xacro" />
+    <xacro:include filename="lidar.xacro" />
+    <xacro:include filename="box.xacro" />
+    <xacro:box parent="base_footprint">
+        <origin xyz="0.0 0 0.0" rpy="0 0 0"/>
+    </xacro:box>
+    <xacro:camera_base parent="base_footprint">
+        <origin xyz="0.0 0.0 0.06" rpy="0.0 0.0 0.0"/>
+    </xacro:camera_base>
+    <xacro:lidar parent="base_footprint">
+        <origin xyz="0.0 0.0 0.11" rpy="0.0 0.0 0.0"/>
+    </xacro:lidar>
 </robot>

File: description/soporte_core.xacro (robot description, xacro)
@@ -23,12 +23,12 @@
             <origin xyz="0.0 0.0 0.0" rpy="0.0 0.0 0.0"/>
             <geometry>
-                <mesh filename="package://perception_system_v2/meshes/soporte_hexag.dae"/>
+                <mesh filename="package://perception_system_v2/meshes/base.dae"/>
             </geometry>
             <material name="white"/>
         </visual>
         <collision>
-            <origin xyz="0.0 0.0 0.0" rpy="0.0 0.0 0.0"/>
+            <origin xyz="0 0.0 0.0" rpy="0.0 0.0 0.0"/>
             <geometry>
-                <mesh filename="package://perception_system_v2/meshes/soporte_hexag.dae"/>
+                <mesh filename="package://perception_system_v2/meshes/base.dae"/>
             </geometry>
         </collision>
@@ -38,27 +38,3 @@
         </xacro:inertial_box>
     </link>
-    <joint name="c1_joint" type="fixed">
-        <origin xyz="0.08660 0.0 0.0" rpy="0.0 0.0 0.0"/>
-        <parent link="base_chassis"/>
-        <child link="oak1-d-base-frame"/>
-    </joint>
-    <link name="oak1-d-base-frame"></link>
-    <joint name="c2_joint" type="fixed">
-        <origin xyz="0.04330 0.075 0.0" rpy="0.0 0.0 ${60*pi/180}"/>
-        <parent link="base_chassis"/>
-        <child link="oak2-d-base-frame"/>
-    </joint>
-    <link name="oak2-d-base-frame"></link>
-    <joint name="c3_joint" type="fixed">
-        <origin xyz="0.04330 -0.075 0.0" rpy="0.0 0.0 ${300*pi/180}"/>
-        <parent link="base_chassis"/>
-        <child link="oak3-d-base-frame"/>
-    </joint>
-    <link name="oak3-d-base-frame"></link>
-    <joint name="c4_joint" type="fixed">
-        <origin xyz="-1.0 0.0 0.0" rpy="0.0 0.0 ${pi}"/>
-        <parent link="base_chassis"/>
-        <child link="oak4-d-base-frame"/>
-    </joint>
-    <link name="oak4-d-base-frame"></link>
 </robot>
