Commit message: minor changes
Signed-off-by: adrianCo <adrian.cobo.mh@gmail.com>

File: description/box.xacro (robot description, xacro)
@@ -15,5 +15,5 @@
                 <origin xyz="-0.065 0.0 0.0" rpy="0.0 0.0 0.0"/>
                 <geometry>
-                    <mesh filename="package://perception_system/meshes/box.dae"/>
+                    <mesh filename="package://perception_system_v2/meshes/box.dae"/>
                 </geometry>
                 <material name="orange"/> <!-- ToDo paint .dae-->
@@ -22,5 +22,5 @@
                 <origin xyz="-0.065 0.0 0.0" rpy="0.0 0.0 0.0"/>
                 <geometry>
-                    <mesh filename="package://perception_system/meshes/box.dae"/>
+                    <mesh filename="package://perception_system_v2/meshes/box.dae"/>
                 </geometry>
             </collision>
